File: hardware/max31855k.kicad_sch (KiCad schematic)
At the start: 6 parts, among them U2 MAX31855KASA

Commit message: chore(hw): migrate KiCad files to the KiCad 10 format
Via `kicad-cli sch upgrade` / `pcb upgrade` (bread-infra
scripts/upgrade_kicad10.sh). Verified lossless: identical netlist, footprint
positions and routing.

Note `sch upgrade` does not cascade into hierarchical sub-sheets, so every
.kicad_sch is upgraded individually -- upgrading only the root sheet leaves
sub-sheets on the old format, which looks migrated and is not.
Parts:
- renumbered C5 to C6, FB1 to FB3, FB2 to FB4, R3 to R5, R4 to R6, U2 to U3
