File: hardware/BREAD_Slice.kicad_pcb (KiCad board)
At the start: 2 copper layers, 70 x 100 mm, 46 parts, among them J1 I2C_01x04, J10 Term_PressFit_1x01_5mm_Phoeni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, J11 Term_PressFit_1x01_5mm_Phoeni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, J12 Term_PressFit_1x01_5mm_Phoeni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, J13 Term_PressFit_1x01_5mm_Phoeni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, J14 Term_PressFit_1x01_5mm_Phoeni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, J2 Conn_01x10_Female, J3 Term_PressFit_1x01_5mm_Phoeni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, J4 Term_PressFit_1x01_5mm_Phoeni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, J5 Term_PressFit_1x01_5mm_Phoeni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, J6 Term_PressFit_1x01_5mm_Phoeni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, J7 Term_PressFit_1x01_5mm_Phoeni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, J8 Term_PressFit_1x01_5mm_Phoeni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, J9 Term_PressFit_1x01_5mm_Phoeni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, Q1 TIP120, Q2 TIP120, Q3 TIP120, Q4 TIP120, U2 MAX31855KASA, U3 MAX31855KASA

Commit message: fix(hw): re-point stale library nicknames
These parts exist in KiCad-Master-Lib; the boards referenced libraries that no
longer exist (kml-custom, KML-Custom, and SparkFun libraries that never
contained the part) or names the library has since changed.

KiCad embeds footprint geometry in the .kicad_pcb, so the boards rendered and
fabricated correctly and the rot stayed invisible -- it only surfaces on
update-from-library, or when a generator tries to resolve a nickname.

Nickname/name only. No geometry is changed:

  KML-Custom:1751066 -> KMLib_Connectors:1751066
  KML-Custom:Thermal Pad -> KMLib_Mounting:Thermal_Pad
  SparkFun-DiscreteSemi:AP63205 -> KMLib_IC_Power:AP63205WU-7_Buck_Regulator
  SparkFun-LED:WS2812-5050-4PIN -> KMLib_IC_SMD:WS2812-5050-4PIN

Only references that failed to resolve were touched. Generic parts (<=4 pins)
and KiCad *-rescue libraries are deliberately excluded: fingerprint matching
cannot distinguish a 2-pin resistor from a 2-pin capacitor, so those are being
done by hand.
Parts:
- D1: footprint SparkFun-LED:WS2812-5050-4PIN -> KMLib_IC_SMD:WS2812-5050-4PIN
- HS1: footprint KML-Custom:Thermal Pad -> KMLib_Mounting:Thermal_Pad
- J10, J11, J12, J13, J14, J3, J4, J5, J6, J7, J8, J9: footprint KML-Custom:1751066 -> KMLib_Connectors:1751066
Changed lines of the file:
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@@
 		(embedded_fonts no)
 	)
-	(footprint "KML-Custom:Thermal Pad"
+	(footprint "KMLib_Mounting:Thermal_Pad"
 		(layer "F.Cu")
 		(at 131.35 121.355)
@@
 		(embedded_fonts no)
 	)
-	(footprint "KML-Custom:1751066"
+	(footprint "KMLib_Connectors:1751066"
 		(layer "F.Cu")
 		(at 188.03 106.51 90)
@@
 		)
 	)
-	(footprint "KML-Custom:1751066"
+	(footprint "KMLib_Connectors:1751066"
 		(layer "F.Cu")
 		(at 187.9 70.4 90)
@@
 		)
 	)
-	(footprint "KML-Custom:1751066"
+	(footprint "KMLib_Connectors:1751066"
 		(layer "F.Cu")
 		(at 188.03 102.11 90)
@@
 		)
 	)
-	(footprint "KML-Custom:1751066"
+	(footprint "KMLib_Connectors:1751066"
 		(layer "F.Cu")
 		(at 188.03 97.71 90)
@@
 		)
 	)
-	(footprint "KML-Custom:1751066"
+	(footprint "KMLib_Connectors:1751066"
 		(layer "F.Cu")
 		(at 188.03 88.91 90)
@@
 		)
 	)
-	(footprint "KML-Custom:1751066"
+	(footprint "KMLib_Connectors:1751066"
 		(layer "F.Cu")
 		(at 188.03 93.31 90)
@@
 		)
 	)
-	(footprint "SparkFun-LED:WS2812-5050-4PIN"
+	(footprint "KMLib_IC_SMD:WS2812-5050-4PIN"
 		(locked yes)
 		(layer "F.Cu")
@@
 		(embedded_fonts no)
 	)
-	(footprint "KML-Custom:1751066"
+	(footprint "KMLib_Connectors:1751066"
 		(layer "F.Cu")
 		(at 187.9 66 90)
@@
 		)
 	)
-	(footprint "KML-Custom:1751066"
+	(footprint "KMLib_Connectors:1751066"
 		(layer "F.Cu")
 		(at 188.03 84.51 90)
@@
 		)
 	)
-	(footprint "KML-Custom:1751066"
+	(footprint "KMLib_Connectors:1751066"
 		(layer "F.Cu")
 		(at 188.03 115.31 90)
@@
 		)
 	)
-	(footprint "KML-Custom:1751066"
+	(footprint "KMLib_Connectors:1751066"
 		(layer "F.Cu")
 		(at 187.9 57.2 90)
@@
 		)
 	)
-	(footprint "KML-Custom:1751066"
+	(footprint "KMLib_Connectors:1751066"
 		(layer "F.Cu")
 		(at 188.03 110.91 90)
@@
 		)
 	)
-	(footprint "KML-Custom:1751066"
+	(footprint "KMLib_Connectors:1751066"
 		(layer "F.Cu")
 		(at 187.9 61.6 90)
