File: hardware/BREAD_Slice.kicad_sch (KiCad schematic)
At the start: 33 parts, among them J1 I2C_01x04, J10 Term_PressFit_1x01_5mm_Phoeni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, J11 Term_PressFit_1x01_5mm_Phoeni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, J12 Term_PressFit_1x01_5mm_Phoeni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, J13 Term_PressFit_1x01_5mm_Phoeni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, J14 Term_PressFit_1x01_5mm_Phoeni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, J2 Conn_01x10_Female, J3 Term_PressFit_1x01_5mm_Phoeni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, J4 Term_PressFit_1x01_5mm_Phoeni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, J5 Term_PressFit_1x01_5mm_Phoeni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, J6 Term_PressFit_1x01_5mm_Phoeni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, J7 Term_PressFit_1x01_5mm_Phoeni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, J8 Term_PressFit_1x01_5mm_Phoeni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, J9 Term_PressFit_1x01_5mm_Phoeni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, Q1 TIP120, Q2 TIP120, Q3 TIP120, Q4 TIP120

Commit message: chore(hw): migrate KiCad files to the KiCad 10 format
Via `kicad-cli sch upgrade` / `pcb upgrade` (bread-infra
scripts/upgrade_kicad10.sh). Verified lossless: identical netlist, footprint
positions and routing.

Note `sch upgrade` does not cascade into hierarchical sub-sheets, so every
.kicad_sch is upgraded individually -- upgrading only the root sheet leaves
sub-sheets on the old format, which looks migrated and is not.
Parts:
- U1: value ~ -> (none)

Commit message: fix(hw): re-point stale library nicknames
These parts exist in KiCad-Master-Lib; the boards referenced libraries that no
longer exist (kml-custom, KML-Custom, and SparkFun libraries that never
contained the part) or names the library has since changed.

KiCad embeds footprint geometry in the .kicad_pcb, so the boards rendered and
fabricated correctly and the rot stayed invisible -- it only surfaces on
update-from-library, or when a generator tries to resolve a nickname.

Nickname/name only. No geometry is changed:

  KML-Custom:1751066 -> KMLib_Connectors:1751066
  KML-Custom:Thermal Pad -> KMLib_Mounting:Thermal_Pad
  SparkFun-DiscreteSemi:AP63205 -> KMLib_IC_Power:AP63205WU-7_Buck_Regulator
  SparkFun-LED:WS2812-5050-4PIN -> KMLib_IC_SMD:WS2812-5050-4PIN

Only references that failed to resolve were touched. Generic parts (<=4 pins)
and KiCad *-rescue libraries are deliberately excluded: fingerprint matching
cannot distinguish a 2-pin resistor from a 2-pin capacitor, so those are being
done by hand.
Parts:
- D1: footprint SparkFun-LED:WS2812-5050-4PIN -> KMLib_IC_SMD:WS2812-5050-4PIN
- HS1: footprint KML-Custom:Thermal Pad -> KMLib_Mounting:Thermal_Pad
- U1: symbol SparkFun-DiscreteSemi:AP63205 -> KMLib_IC_Power:AP63205WU-7_Buck_Regulator
Changed lines of the file:
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@@
 	)
 	(symbol
-		(lib_id "SparkFun-DiscreteSemi:AP63205")
+		(lib_id "KMLib_IC_Power:AP63205WU-7_Buck_Regulator")
 		(at 31.75 96.52 0)
 		(unit 1)
@@
 			)
 		)
-		(property "Footprint" "KML-Custom:Thermal Pad"
+		(property "Footprint" "KMLib_Mounting:Thermal_Pad"
 			(at 45.72 112.0648 0)
 			(hide yes)
@@
 			)
 		)
-		(property "Footprint" "SparkFun-LED:WS2812-5050-4PIN"
+		(property "Footprint" "KMLib_IC_SMD:WS2812-5050-4PIN"
 			(at 49.53 76.2 0)
 			(hide yes)
