File: hardware/BREAD_Slice.kicad_sch (KiCad schematic)
At the start: 33 parts, among them J1 I2C_01x04, J10 Term_PressFit_1x01_5mm_Phoeni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, J11 Term_PressFit_1x01_5mm_Phoeni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, J12 Term_PressFit_1x01_5mm_Phoeni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, J13 Term_PressFit_1x01_5mm_Phoeni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, J14 Term_PressFit_1x01_5mm_Phoeni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, J2 Conn_01x10_Female, J3 Term_PressFit_1x01_5mm_Phoeni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, J4 Term_PressFit_1x01_5mm_Phoeni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, J5 Term_PressFit_1x01_5mm_Phoeni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, J6 Term_PressFit_1x01_5mm_Phoeni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, J7 Term_PressFit_1x01_5mm_Phoeni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, J8 Term_PressFit_1x01_5mm_Phoeni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, J9 Term_PressFit_1x01_5mm_Phoeni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, Q1 TIP120, Q2 TIP120, Q3 TIP120, Q4 TIP120

Commit message: fix(hw): restore library prefixes on schematic Footprint properties
A symbol's Footprint property must be "Library:Item". These carried only the bare
item name, so KiCad reported a schematic/PCB parity error:

    KMLib_Connectors:1439890 doesn't match footprint given by symbol (1439890)

The prefix is taken from the PCB, which holds the full lib_id, matched by
reference designator -- not guessed. Symbols whose reference is absent from the
PCB, or whose PCB footprint has a different item name, were left alone.

No geometry changes; only the Footprint property text.

Schematic parity errors: 12 -> 0
Parts:
- J10, J11, J12, J13, J14, J3, J4, J5, J6, J7, J8, J9: footprint 1751066 -> KMLib_Connectors:1751066
Changed lines of the file:
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@@
 			)
 		)
-		(property "Footprint" "1751066"
+		(property "Footprint" "KMLib_Connectors:1751066"
 			(at 166.37 178.74 0)
 			(hide yes)
@@
 			)
 		)
-		(property "Footprint" "1751066"
+		(property "Footprint" "KMLib_Connectors:1751066"
 			(at 243.84 158.42 0)
 			(hide yes)
@@
 			)
 		)
-		(property "Footprint" "1751066"
+		(property "Footprint" "KMLib_Connectors:1751066"
 			(at 143.51 192.71 0)
 			(hide yes)
@@
 			)
 		)
-		(property "Footprint" "1751066"
+		(property "Footprint" "KMLib_Connectors:1751066"
 			(at 166.37 167.31 0)
 			(hide yes)
@@
 			)
 		)
-		(property "Footprint" "1751066"
+		(property "Footprint" "KMLib_Connectors:1751066"
 			(at 139.7 133.02 0)
 			(hide yes)
@@
 			)
 		)
-		(property "Footprint" "1751066"
+		(property "Footprint" "KMLib_Connectors:1751066"
 			(at 246.38 223.19 0)
 			(hide yes)
@@
 			)
 		)
-		(property "Footprint" "1751066"
+		(property "Footprint" "KMLib_Connectors:1751066"
 			(at 144.78 204.14 0)
 			(hide yes)
@@
 			)
 		)
-		(property "Footprint" "1751066"
+		(property "Footprint" "KMLib_Connectors:1751066"
 			(at 139.7 121.59 0)
 			(hide yes)
@@
 			)
 		)
-		(property "Footprint" "1751066"
+		(property "Footprint" "KMLib_Connectors:1751066"
 			(at 168.91 256.21 0)
 			(hide yes)
@@
 			)
 		)
-		(property "Footprint" "1751066"
+		(property "Footprint" "KMLib_Connectors:1751066"
 			(at 246.38 230.81 0)
 			(hide yes)
@@
 			)
 		)
-		(property "Footprint" "1751066"
+		(property "Footprint" "KMLib_Connectors:1751066"
 			(at 168.91 244.78 0)
 			(hide yes)
@@
 			)
 		)
-		(property "Footprint" "1751066"
+		(property "Footprint" "KMLib_Connectors:1751066"
 			(at 243.84 150.8 0)
 			(hide yes)
